File: ground_station/pcb/ground_station.kicad_sch (KiCad schematic)
At the start: 25 parts, among them J1 Conn_01x02_Pin, J10 Conn_01x11_Socket, J11 Conn_01x02_Socket, J12 Conn_01x04_Socket, J13 Conn_01x02_Socket, J2 Conn_01x03_Pin, J3 Conn_01x08_Socket, J4 Conn_01x06_Pin, J5 Conn_01x06_Pin, J6 Conn_01x02_Socket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

Commit message: Completed tracing work
Parts:
- removed D1: LED_BGAR, LED_THT:LED_D5.0mm-4_RGB, symbol Device:LED_BGAR
- removed J10: Conn_01x11_Socket, Connector_PinSocket_2.54mm:PinSocket_1x11_P2.54mm_Vertical, symbol Connector:Conn_01x11_Socket
- added J10: Conn_01x13_Socket, Connector_PinSocket_2.54mm:PinSocket_1x13_P2.54mm_Vertical, symbol Connector:Conn_01x13_Socket
- added J14: Conn_01x04_Socket, Connector_PinSocket_2.54mm:PinSocket_1x04_P2.54mm_Vertical, symbol Connector:Conn_01x04_Socket
- H1, H2, H3, H4: footprint MountingHole:MountingHole_2.2mm_M2 -> MountingHole:MountingHole_2.5mm
Connections:
- net +3.3V: now also J6.2 (Pin_2)
- net A0: now also J10.12 (Pin_12)
- net A3: now also J10.11 (Pin_11)
- net D11: now also J10.8 (Pin_8); no longer J6.2 (Pin_2)
- net D13: now also J10.6 (Pin_6)
- net D25: now also J10.9 (Pin_9)
- net EN: now also J10.10 (Pin_10)
- net GND: now also J10.7 (Pin_7), J14.2 (Pin_2)
- net MISO: now also J10.3 (Pin_3)
- net MOSI: now also J10.4 (Pin_4)
- net RESET: now also J10.13 (Pin_13)
- net RX: now also J10.2 (Pin_2)
- net SCK: now also J10.5 (Pin_5)
- net TX: now also J10.1 (Pin_1)
- net BL_IN: now reaches R4.2
- net BL_IN: now also J14.4 (Pin_4)
- net GRN_IN: now reaches R3.2
- net GRN_IN: now also J14.3 (Pin_3)
- net RED_IN: now reaches R2.2
- net RED_IN: now also J14.1 (Pin_1)
Other:
- note added: "2.5mm Size Mounting Holes"
- note added: "BLUE"
- note added: "GREEN"
- note added: "RED"
- note removed: "M2 Size (2.2mm) Mounting Holes"
