File: ground_station/pcb/ground_station.kicad_pcb (KiCad board)
At the start: 2 copper layers, 102 x 70 mm, 25 parts, among them J1 Conn_01x02_Pin, J10 Conn_01x11_Socket, J11 Conn_01x02_Socket, J12 Conn_01x04_Socket, J13 Conn_01x02_Socket, J2 Conn_01x03_Pin, J3 Conn_01x08_Socket, J4 Conn_01x06_Pin, J5 Conn_01x06_Pin, J6 Conn_01x02_Socket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

Commit message: Completed tracing work
Parts:
- removed D1: LED_BGAR, LED_THT:LED_D5.0mm-4_RGB
- added G***: LOGO, graphics:rocket_logo_black_48_no_window, F.Cu at (127.7, 59.5)
- added J14: Conn_01x04_Socket, Connector_PinSocket_2.54mm:PinSocket_1x04_P2.54mm_Vertical, F.Cu at (180.8, 60.7)
- H1, H2, H3, H4: footprint MountingHole:MountingHole_2.2mm_M2 -> MountingHole:MountingHole_2.5mm
- J10: value Conn_01x11_Socket -> Conn_01x13_Socket; footprint Connector_PinSocket_2.54mm:PinSocket_1x11_P2.54mm_Vertical -> Connector_PinSocket_2.54mm:PinSocket_1x13_P2.54mm_Vertical
- moved H1 18.0 mm to (82.2, 120.8)
- moved H3 18.0 mm to (82.2, 56.8)
- moved J12 11.8 mm to (102.3, 98.2)
- moved J7 8.52 mm to (104.0, 116.5)
- moved J10 6.58 mm to (196.3, 73.3)
- moved J3 4.48 mm to (114.0, 78.6), turned to 180 degrees
- moved R4 4.29 mm to (178.4, 81.8)
- moved R3 2.55 mm to (178.4, 74.9)
- moved R2 1.92 mm to (178.4, 68.2)
- moved J11 0.17 mm to (196.3, 110.9)
- moved R1 0.06 mm to (186.4, 114.7)
Connections:
- J10 pad 1: /RESET -> /TX
- J10 pad 10: /D24 -> /EN
- J10 pad 11: /A0 -> /A3
- J10 pad 2: /EN -> /RX
- J10 pad 3: /TX -> /MISO
- J10 pad 4: /RX -> /MOSI
- J10 pad 5: /MISO -> /SCK
- J10 pad 6: /MOSI -> /D13
- J10 pad 7: /SCK -> GND
- J10 pad 8: /A3 -> /D11
- J10 pad 9: /D13 -> /D25
- J6 pad 2: /D11 -> +3.3V
- R2 pad 2: Net-(D1-RK) -> /RED_IN
- R3 pad 2: Net-(D1-GK) -> /GRN_IN
- R4 pad 2: Net-(D1-BK) -> /BL_IN
Routing:
- net +3.3V: track 0.00 -> 178.2 mm
- net /SDA: track 0.00 -> 75.7 mm
- net /SCL: track 0.00 -> 72.1 mm
- net /D10: track 0.00 -> 55.7 mm, vias 0 -> 2
- net /D13: track 0.00 -> 55.5 mm, vias 0 -> 4
- net /EN: track 0.00 -> 51.5 mm
- net /D11: track 0.00 -> 48.9 mm
- net GND: track 0.00 -> 41.6 mm, vias 0 -> 8
- net /RESET: track 0.00 -> 40.1 mm, vias 0 -> 2
- net /D9: track 0.00 -> 36.5 mm
- net /D5: track 0.00 -> 36.3 mm
- net /D12: track 0.00 -> 34.8 mm, vias 0 -> 2
- net /D6: track 0.00 -> 34.5 mm
- net /TX: track 0.00 -> 33.0 mm
- net /RX: track 0.00 -> 32.3 mm
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- added copper zone on B.Cu, net GND
Other:
- board size 102 x 70 mm -> 120 x 70 mm
- board text added: "3.3V"
- board text added: "A0"
- board text added: "A1"
- board text added: "A2"
- board text added: "A3"
- board text added: "AHT20"
- board text added: "B"
- board text added: "BAT"
- board text added: "BMP390"
- board text added: "Big Red Btn"
- board text added: "Chris Silman Colin McKinney Chase Engle Collin Hoffman Cole Thornton Brandon Crudele William Li"
- board text added: "D10"
- board text added: "D11"
- board text added: "D12"
- board text added: "D13"
- board text added: "D24"
- board text added: "D25"
- board text added: "Designed by:"
- board text added: "ECE56800 Ground Station"
- board text added: "EN"
- board text added: "Encoder"
- board text added: "Feather RP2040 RFM95"
- board text added: "G"
- board text added: "GND"
- board text added: "Key Switch"
- board text added: "LED"
- board text added: "MISO"
- board text added: "MOSI"
- board text added: "MiniGPS"
- board text added: "R"
- board text added: "RST"
- board text added: "Rx"
- board text added: "SCK"
- board text added: "SCL"
- board text added: "SDA"
- board text added: "Tx"
- board text added: "USB 5V"

Commit message: Pushed manufacturing files
Routing:
- net GND: track 41.6 -> 57.8 mm, vias 8 -> 11
Changed lines of the file:
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@@
 			(usegerberattributes yes)
 			(usegerberadvancedattributes yes)
-			(creategerberjobfile yes)
+			(creategerberjobfile no)
 			(dashed_line_dash_ratio 12.000000)
 			(dashed_line_gap_ratio 3.000000)
@@
 			(outputformat 1)
 			(mirror no)
-			(drillshape 1)
+			(drillshape 0)
 			(scaleselection 1)
-			(outputdirectory "")
+			(outputdirectory "Manufacturing/")
 		)
 	)
@@
 		)
 		(property "Value" "Conn_01x02_Socket"
-			(at 0 5.31 0)
+			(at 1.2 -1.66 0)
 			(layer "F.Fab")
 			(effects
@@
 		)
 		(property "Value" "Conn_01x04_Socket"
-			(at -1.2 7.39 0)
+			(at -0.9 10.18 0)
 			(layer "F.Fab")
 			(effects
@@
 	)
 	(segment
+		(start 183.36 59.46)
+		(end 182.5 58.6)
+		(width 0.7)
+		(layer "F.Cu")
+		(net 3)
+	)
+	(segment
 		(start 186.4 114.74)
 		(end 184.24 114.74)
@@
 	)
 	(segment
+		(start 183.36 60.675)
+		(end 183.36 59.46)
+		(width 0.7)
+		(layer "F.Cu")
+		(net 3)
+	)
+	(segment
 		(start 111.44 116.54)
 		(end 111.4 116.5)
@@
 	)
 	(segment
+		(start 141.2 91.38)
+		(end 144.18 91.38)
+		(width 0.7)
+		(layer "F.Cu")
+		(net 3)
+	)
+	(segment
+		(start 144.18 91.38)
+		(end 144.2 91.4)
+		(width 0.7)
+		(layer "F.Cu")
+		(net 3)
+	)
+	(segment
+		(start 141.6 118.54)
+		(end 144.86 118.54)
+		(width 0.7)
+		(layer "F.Cu")
+		(net 3)
+	)
+	(segment
 		(start 196.3 88.5)
 		(end 194.7 88.5)
@@
 	)
 	(segment
+		(start 144.86 118.54)
+		(end 144.9 118.5)
+		(width 0.7)
+		(layer "F.Cu")
+		(net 3)
+	)
+	(segment
 		(start 113.8 116.54)
 		(end 111.44 116.54)
@@
 	)
 	(segment
+		(start 134.2 118.54)
+		(end 141.6 118.54)
+		(width 0.7)
+		(layer "F.Cu")
+		(net 3)
+	)
+	(segment
 		(start 165.53 109.43)
 		(end 165.5 109.4)
@@
 	)
 	(via
+		(at 144.9 118.5)
+		(size 0.8)
+		(drill 0.4)
+		(layers "F.Cu" "B.Cu")
+		(net 3)
+	)
+	(via
 		(at 165.5 109.4)
 		(size 0.8)
@@
 	)
 	(via
+		(at 144.2 91.4)
+		(size 0.8)
+		(drill 0.4)
+		(layers "F.Cu" "B.Cu")
+		(net 3)
+	)
+	(via
 		(at 124.3 116.5)
 		(size 0.8)
@@
 		(size 0.8)
 		(drill 0.4)
+		(layers "F.Cu" "B.Cu")
+		(net 3)
+	)
+	(via
+		(at 182.5 58.6)
+		(size 0.8)
+		(drill 0.4)
